File: Low_Pass_Filter.kicad_sch (KiCad schematic)
At the start: 7 parts

Commit message: Commit just prior to pushing to Github.  Design not complete.
Parts:
- renumbered C57 to C14, C58 to C15, C59 to C43, C60 to C44, L15 to L3, L16 to L4, L17 to L5
Changed lines of the file:
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@@
 (kicad_sch
-	(version 20231120)
+	(version 20250114)
 	(generator "eeschema")
-	(generator_version "8.0")
+	(generator_version "9.0")
 	(paper "A4")
 	(junction
@@
 		(shape output)
 		(at 165.1 87.63 0)
-		(fields_autoplaced yes)
 		(effects
 			(font
@@
 		(shape input)
 		(at 114.3 87.63 180)
-		(fields_autoplaced yes)
 		(effects
 			(font
@@
 		(dnp no)
 		(fields_autoplaced yes)
-		(property "Reference" "L15"
+		(property "Reference" "L3"
 			(at 127 82.55 90)
 			(effects
@@
 		(on_board yes)
 		(dnp no)
-		(property "Reference" "C57"
+		(property "Reference" "C14"
 			(at 123.19 91.44 0)
 			(effects
@@
 		(dnp no)
 		(fields_autoplaced yes)
-		(property "Reference" "L16"
+		(property "Reference" "L4"
 			(at 138.43 82.55 90)
 			(effects
@@
 		(dnp no)
 		(fields_autoplaced yes)
-		(property "Reference" "L17"
+		(property "Reference" "L5"
 			(at 149.86 82.55 90)
 			(effects
@@
 		(on_board yes)
 		(dnp no)
-		(property "Reference" "#PWR049"
+		(property "Reference" "#PWR07"
 			(at 137.16 105.41 0)
 			(effects
@@
 		(dnp no)
 		(fields_autoplaced yes)
-		(property "Reference" "C59"
+		(property "Reference" "C43"
 			(at 146.05 91.4335 0)
 			(effects
@@
 		(dnp no)
 		(fields_autoplaced yes)
-		(property "Reference" "C60"
+		(property "Reference" "C44"
 			(at 157.48 91.4335 0)
 			(effects
@@
 		(dnp no)
 		(fields_autoplaced yes)
-		(property "Reference" "C58"
+		(property "Reference" "C15"
 			(at 134.62 91.4335 0)
 			(effects

Commit message: Trying to improve schematic by adding capacitor values to all bands.
Parts:
- C14: value 470pF -> ${C_1}
Changed lines of the file:
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@@
 			)
 		)
-		(property "Value" "470pF"
+		(property "Value" "${C_1}"
 			(at 123.19 93.98 0)
 			(effects

Commit message: T41-2 LPF V1.4 to fab.
Parts:
- C14: value ${C_1} -> ${C1}
- C15: value 1200pF -> ${C2}
- C43: value 1200pF -> ${C3}
- C44: value 470pF -> ${C4}
Changed lines of the file:
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@@
 		)
 		(instances
-			(project "t41_2_lpf_board_orthog"
+			(project "T41_2_lpf"
 				(path "/5fc700c6-272f-41b7-8650-23a96fb06ce8/25f7731c-bad8-4554-9b01-13138334dc1b"
 					(reference "L15")
@@
 			)
 		)
-		(property "Value" "${C_1}"
+		(property "Value" "${C1}"
 			(at 123.19 93.98 0)
 			(effects
@@
 		)
 		(instances
-			(project "t41_2_lpf_board_orthog"
+			(project "T41_2_lpf"
 				(path "/5fc700c6-272f-41b7-8650-23a96fb06ce8/25f7731c-bad8-4554-9b01-13138334dc1b"
 					(reference "C57")
@@
 		)
 		(instances
-			(project "t41_2_lpf_board_orthog"
+			(project "T41_2_lpf"
 				(path "/5fc700c6-272f-41b7-8650-23a96fb06ce8/25f7731c-bad8-4554-9b01-13138334dc1b"
 					(reference "L16")
@@
 		)
 		(instances
-			(project "t41_2_lpf_board_orthog"
+			(project "T41_2_lpf"
 				(path "/5fc700c6-272f-41b7-8650-23a96fb06ce8/25f7731c-bad8-4554-9b01-13138334dc1b"
 					(reference "L17")
@@
 		)
 		(instances
-			(project "t41_2_lpf_board_orthog"
+			(project "T41_2_lpf"
 				(path "/5fc700c6-272f-41b7-8650-23a96fb06ce8/25f7731c-bad8-4554-9b01-13138334dc1b"
 					(reference "#PWR049")
@@
 			)
 		)
-		(property "Value" "1200pF"
+		(property "Value" "${C3}"
 			(at 146.05 93.9735 0)
 			(effects
@@
 		)
 		(instances
-			(project "t41_2_lpf_board_orthog"
+			(project "T41_2_lpf"
 				(path "/5fc700c6-272f-41b7-8650-23a96fb06ce8/25f7731c-bad8-4554-9b01-13138334dc1b"
 					(reference "C59")
@@
 			)
 		)
-		(property "Value" "470pF"
+		(property "Value" "${C4}"
 			(at 157.48 93.9735 0)
 			(effects
@@
 		)
 		(instances
-			(project "t41_2_lpf_board_orthog"
+			(project "T41_2_lpf"
 				(path "/5fc700c6-272f-41b7-8650-23a96fb06ce8/25f7731c-bad8-4554-9b01-13138334dc1b"
 					(reference "C60")
@@
 			)
 		)
-		(property "Value" "1200pF"
+		(property "Value" "${C2}"
 			(at 134.62 93.9735 0)
 			(effects
@@
 		)
 		(instances
-			(project "t41_2_lpf_board_orthog"
+			(project "T41_2_lpf"
 				(path "/5fc700c6-272f-41b7-8650-23a96fb06ce8/25f7731c-bad8-4554-9b01-13138334dc1b"
 					(reference "C58")

Commit message: Work in progress just prior to publish.
Other:
- note added: "T44-2 TOROIDS"
