File: Low_Pass_Filter.kicad_sch (KiCad schematic)
At the start: 7 parts

Commit message: Schematic clean-up.
Other:
- note removed: "T44-2 TOROIDS"
Changed lines of the file:
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@@
 	(generator_version "10.0")
 	(paper "A4")
-	(text "T44-2 TOROIDS"
-		(exclude_from_sim no)
-		(at 21.9286 14.104 0)
-		(effects
-			(font
-				(size 1.5 1.5)
-				(thickness 0.3)
-				(bold yes)
-			)
-		)
-	)
-	(text "T44-2 TOROIDS"
-		(exclude_from_sim no)
-		(at 15.5786 7.754 0)
-		(effects
-			(font
-				(size 1.5 1.5)
-				(thickness 0.3)
-				(bold yes)
-			)
-		)
-	)
-	(text "T44-2 TOROIDS"
-		(exclude_from_sim no)
-		(at 9.2286 1.404 0)
-		(effects
-			(font
-				(size 1.5 1.5)
-				(thickness 0.3)
-				(bold yes)
-			)
-		)
-	)
 	(junction
 		(at 132.08 97.79)
@@
 		)
 	)
-	(label "16T 13T 16T"
-		(at 7.9586 11.818 0)
-		(effects
-			(font
-				(size 1.5 1.5)
-				(thickness 0.3)
-				(bold yes)
-			)
-			(justify left bottom)
-		)
-	)
-	(label "16T 13T 16T"
-		(at 1.6086 5.468 0)
-		(effects
-			(font
-				(size 1.5 1.5)
-				(thickness 0.3)
-				(bold yes)
-			)
-			(justify left bottom)
-		)
-	)
-	(label "16T 13T 16T"
-		(at 19.35 21.975 0)
-		(effects
-			(font
-				(size 1.5 1.5)
-				(thickness 0.3)
-				(bold yes)
-			)
-			(justify left bottom)
-		)
-	)
-	(label "16T 13T 16T"
-		(at 14.3086 18.168 0)
-		(effects
-			(font
-				(size 1.5 1.5)
-				(thickness 0.3)
-				(bold yes)
-			)
-			(justify left bottom)
-		)
-	)
