File: RelaySwitches.kicad_sch (KiCad schematic)
At the start: 50 parts, among them Q1 Q_NMOS_GSD, Q2 Q_NMOS_GSD, Q3 Q_NMOS_GSD, Q4 Q_NMOS_GSD, Q5 Q_NMOS_GSD

Commit message: Work in progress just prior to publish.
Parts:
- RL1, RL10, RL2, RL3, RL4, RL5, RL6, RL7, RL8, RL9: value ~ -> (none)
