File: T41_2_lpf.kicad_pcb (KiCad board)
At the start: 2 copper layers, 100 x 100 mm, 116 parts, among them J1 5-1814832-1, J2 5-1814832-1, J3 5-1814832-1, J4 Conn_02x08_Odd_Even, J5 Conn_02x05_Odd_Even, J6 B2B-XH-A_LF__SN_, Q1 Q_NMOS_GSD, Q2 Q_NMOS_GSD, Q3 Q_NMOS_GSD, Q4 Q_NMOS_GSD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

Commit message: Ready for fab.
Routing:
- net /12V_RELAY: track 375.3 -> 381.8 mm
- net Net-(Q4-D): track 68.6 -> 70.4 mm
- net Net-(Q3-D): track 71.7 -> 73.4 mm
- net Net-(Q2-D): track 79.7 -> 81.5 mm
- net Net-(Q5-D): track 76.2 -> 77.5 mm
- net GND: vias 211 -> 220
Other:
- board text added: "OPEN HARDWARE"

Commit message: T41-2 LPF V1.4 to fab.
Parts:
- removed C2: 0.1uF, Capacitor_SMD:C_1206_3216Metric
- removed FB12: 28F0121-0SR-10, Inductor_SMD:L_1206_3216Metric
- removed R10: 470, Resistor_SMD:R_1206_3216Metric
- removed R7, R8: 0, Resistor_SMD:R_1206_3216Metric
- removed R9: 4700, Resistor_SMD:R_1206_3216Metric
- added TP1: GND, Connector_PinHeader_2.54mm:PinHeader_1x01_P2.54mm_Vertical, F.Cu at (118.4, 109.2)
- C14, C44: value 470pF -> 1300pF
- C15, C43: value 1200pF -> 3600pF
- C45, C48: value 470pF -> 680pF
- C46, C47: value 1200pF -> 1800pF
- C49, C52: value 470pF -> 270pF
- C50, C51: value 1200pF -> 820pF
- C53, C56: value 470pF -> 180pF
- C54, C55: value 1200pF -> 510pF
- C57, C60: value 470pF -> 150pF
- C58, C59: value 1200pF -> 390pF
Connections:
- FB13 pad 1: /3_3V -> /3_3V_IN
- J4 pad 13: /3_3V -> /3_3V_IN
- J4 pad 14: /3_3V -> /3_3V_IN
- J4 pad 5: /12VIN -> /12V_IN
- J4 pad 6: /12VIN -> /12V_IN
- RL11 pad 8: Net-(R10-Pad2) -> unconnected-(RL11-Pad8)
Routing:
- net /12VIN: track 38.4 -> 0.00 mm
- net /12V_IN: track 30.0 -> 64.3 mm, vias 1 -> 3
- net /3_3V_IN: track 14.5 -> 42.2 mm, vias 0 -> 2
- net /3_3V: track 27.5 -> 0.00 mm
- net Net-(R10-Pad2): track 7.51 -> 0.00 mm
- net Net-(RL1-Pad2): track 17.5 -> 13.1 mm
- net /12V_FIL: track 2.89 -> 0.00 mm
- net /TXRX: track 80.3 -> 79.7 mm
Other:
- board text added: "T41-2 LOW PASS FILTER V1.4"
- board text removed: "T41-2 LOW PASS FILTER V1.3"

Commit message: Ready to fab version 1.5
Parts:
- removed C14, C44: 1300pF, Capacitor_SMD:C_1206_3216Metric
- removed C15, C43: 3600pF, Capacitor_SMD:C_1206_3216Metric
- removed L3, L4, L5: L, Toroid_SMD:Toroid_SMD_Thin
- added C62: 1300pF, Capacitor_SMD:C_1206_3216Metric, F.Cu at (153.3, 131.8)
- added C63: 3600pF, Capacitor_SMD:C_1206_3216Metric, F.Cu at (163.7, 143.7)
- added C64: 3600pF, Capacitor_SMD:C_1206_3216Metric, F.Cu at (170.5, 136.2)
- added C65: 1300pF, Capacitor_SMD:C_1206_3216Metric, F.Cu at (176.2, 132.0)
- added C66: 1300pF, Capacitor_SMD:C_1206_3216Metric, F.Cu at (158.2, 131.8)
- added C67: 3600pF, Capacitor_SMD:C_1206_3216Metric, F.Cu at (163.7, 136.2)
- added C68: 1300pF, Capacitor_SMD:C_1206_3216Metric, F.Cu at (181.0, 132.0)
- added C69: 3600pF, Capacitor_SMD:C_1206_3216Metric, F.Cu at (170.5, 143.7)
- added L18: L, Toroid_SMD:Toroid_SMD_Thin, B.Cu at (157.7, 135.1)
- added L19: L, Toroid_SMD:Toroid_SMD_Thin, B.Cu at (167.1, 140.0)
- added L20: L, Toroid_SMD:Toroid_SMD_Thin, B.Cu at (176.4, 135.1)
- TP1: value GND -> TestPoint
Connections:
- RL10 pad 3: /Filter/Output -> /Filter5/Output
- RL9 pad 8: /Filter/Input -> /Filter5/Input
Routing:
- net Net-(C63-Pad2): track 0.00 -> 15.2 mm, vias 0 -> 2
- net Net-(C64-Pad2): track 0.00 -> 15.1 mm, vias 0 -> 2
- net /Filter5/Output: track 0.00 -> 14.9 mm, vias 0 -> 2
- net /Filter5/Input: track 0.00 -> 14.1 mm, vias 0 -> 2
- net /Filter/Output: track 13.0 -> 0.00 mm, vias 2 -> 0
- net /Filter/Input: track 12.1 -> 0.00 mm, vias 2 -> 0
- net Net-(C15-Pad2): track 10.2 -> 0.00 mm, vias 2 -> 0
- net Net-(C43-Pad2): track 10.1 -> 0.00 mm, vias 2 -> 0
- net GND: vias 220 -> 226
Other:
- board text added: "T41-2 LOW PASS FILTER V1.5"
- board text removed: "OPEN HARDWARE"
- board text removed: "T41-2 LOW PASS FILTER V1.4"
