File: T41_2_lpf.kicad_pcb (KiCad board)
At the start: 2 copper layers, 100 x 100 mm, 115 parts, among them J1 5-1814832-1, J2 5-1814832-1, J3 5-1814832-1, J4 Conn_02x08_Odd_Even, J5 Conn_02x05_Odd_Even, J6 B2B-XH-A_LF__SN_, Q1 Q_NMOS_GSD, Q2 Q_NMOS_GSD, Q3 Q_NMOS_GSD, Q4 Q_NMOS_GSD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

Commit message: Final clean-up.
Parts:
- added R7: 100k, Resistor_SMD:R_1206_3216Metric, F.Cu at (183.0, 55.3)
- C45, C48: value 680pF -> 510pF
- C46, C47: value 1800pF -> 1100pF
- C49, C52: value 270pF -> 300pF
- C50, C51: value 820pF -> 560pF
- C53, C56: value 180pF -> 200pF
- C54, C55: value 510pF -> 360pF
- C58, C59: value 390pF -> 300pF
- C62, C68: value 1300pF -> 430pF
- C63, C69: value 3600pF -> 1500pF
- C64, C67: value 3600pF -> 1000pF
- C65, C66: value 1300pF -> 1000pF
Routing:
- net Net-(C61-Pad1): track 6.28 -> 12.1 mm
