File: Low_Pass_Filter_80M.kicad_sch (KiCad schematic)
At the start: 7 parts

Commit message: Ready to fab version 1.5
Parts:
- added C66: ${C1}, Capacitor_SMD:C_1206_3216Metric, symbol Device:C_Small
- added C67: ${C2}, Capacitor_SMD:C_1206_3216Metric, symbol Device:C_Small
- added C68: ${C4}, Capacitor_SMD:C_1206_3216Metric, symbol Device:C_Small
- added C69: ${C3}, Capacitor_SMD:C_1206_3216Metric, symbol Device:C_Small
- renumbered C45 to C62, C46 to C63, C47 to C64, C48 to C65, L6 to L18, L7 to L19, L8 to L20
Connections:
- net GND: now also C66.1, C67.1, C68.1, C69.1
- net Input: now also C66.2
- net Output: now also C68.2
- net at C63.2, L18.2, L19.1: now also C67.2
- net at C64.2, L19.2, L20.1: now also C69.2
Other:
- note removed: "T44-2 TOROIDS"
- moved on the sheet: C62, C64, C65, L18, L19, L20

Commit message: Schematic clean-up.
Parts:
- C62: value ${C1} -> ${C1b}
- C63: value ${C2} -> ${C2b}
- C68: value ${C4} -> ${C4b}
- C69: value ${C3} -> ${C3b}
Changed lines of the file:
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@@
 			)
 		)
-		(property "Value" "${C1}"
+		(property "Value" "${C1b}"
 			(at 106.68 93.98 0)
 			(show_name no)
@@
 			)
 		)
-		(property "Value" "${C4}"
+		(property "Value" "${C4b}"
 			(at 190.5 93.9735 0)
 			(show_name no)
@@
 			)
 		)
-		(property "Value" "${C3}"
+		(property "Value" "${C3b}"
 			(at 162.306 93.726 0)
 			(show_name no)
@@
 			)
 		)
-		(property "Value" "${C2}"
+		(property "Value" "${C2b}"
 			(at 134.62 93.9735 0)
 			(show_name no)
