File: T41_2_lpf.kicad_sch (KiCad schematic)
At the start: 36 parts, among them J1 5-1814832-1, J2 5-1814832-1, J3 5-1814832-1, J4 Conn_02x08_Odd_Even, J5 Conn_02x05_Odd_Even, J6 B2B-XH-A_LF__SN_, Q6 Q_NMOS_GSD, U12 4002, U13 TCA9534

Commit message: Ready to release V1.5 to fab.
Other:
- note added: "CD4002BM96"
- note added: "JST"
- note added: "SMA connectors can be straight or 90 degree. Use the option which minimizes bends and cable lengths."
Changed lines of the file:
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@@
 		(rev "V1.5")
 	)
+	(text "SMA connectors can be straight or 90 degree.\nUse the option which minimizes bends and cable lengths."
+		(exclude_from_sim no)
+		(at 46.99 32.766 0)
+		(effects
+			(font
+				(size 1.5 1.5)
+				(thickness 0.254)
+				(bold yes)
+			)
+		)
+	)
 	(text "TO RECEIVER"
 		(exclude_from_sim no)
@@
 	(text "T44-2 TOROIDS"
 		(exclude_from_sim no)
-		(at 188.976 141.478 0)
+		(at 189.23 146.558 0)
 		(effects
 			(font
@@
 		)
 	)
+	(text "CD4002BM96"
+		(exclude_from_sim no)
+		(at 118.364 196.342 0)
+		(effects
+			(font
+				(size 2 2)
+				(thickness 0.4)
+				(bold yes)
+			)
+		)
+	)
 	(text "PANASONIC\n RELAYS"
 		(exclude_from_sim no)
@@
 				(bold yes)
 			)
+		)
+	)
+	(text "JST"
+		(exclude_from_sim no)
+		(at 57.15 149.86 0)
+		(effects
+			(font
+				(size 1.5 1.5)
+				(thickness 0.3)
+				(bold yes)
+			)

Commit message: Schematic clean-up.
Other:
- note added: "10 TURNS #24"
- note added: "12 TURNS #24"
- note added: "17 TURNS #24"
- note added: "18 TURNS #24"
- note added: "8 TURNS #24"
- note added: "All filters are "Uni-Coil", with the same number of turns on all 3 toroids."
- note added: "PLEASE NOTE THIS RELAY IS ROTATED 180 DEGREES COMPARED TO THE BAND SWITCHING RELAYS!"
- note added: "RECEIVER PATH HIGH-PASS FILTER"
- note added: "T41-2 LOW PASS FILTER BOARD"
- note removed: "T41-2 LOW PASS FILTER"
- moved on the sheet: TP1

Commit message: Final clean-up.
Parts:
- added R7: 100k, Resistor_SMD:R_1206_3216Metric, symbol Device:R_Small_US
Connections:
- net GND: now also R7.1
- net at C61.1, J3.2: now also R7.2
Changed lines of the file:
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@@
 	(text "ANTENNA"
 		(exclude_from_sim no)
-		(at 254 38.1 0)
+		(at 256.54 37.846 0)
 		(effects
 			(font
@@
 	)
 	(junction
+		(at 245.11 22.86)
+		(diameter 0)
+		(color 0 0 0 0)
+	)
+	(junction
 		(at 148.59 78.74)
 		(diameter 0)
@@
 	(wire
 		(pts
-			(xy 241.3 22.86) (xy 248.92 22.86)
+			(xy 241.3 22.86) (xy 245.11 22.86)
 		)
 		(stroke
@@
 	(wire
 		(pts
+			(xy 245.11 30.48) (xy 245.11 31.75)
+		)
+		(stroke
+			(width 0)
+			(type default)
+		)
+	)
+	(wire
+		(pts
 			(xy 214.63 124.46) (xy 209.55 124.46)
 		)
@@
 	(wire
 		(pts
+			(xy 245.11 22.86) (xy 248.92 22.86)
+		)
+		(stroke
+			(width 0)
+			(type default)
+		)
+	)
+	(wire
+		(pts
 			(xy 163.83 115.57) (xy 157.48 115.57)
 		)
@@
 	(wire
 		(pts
+			(xy 245.11 22.86) (xy 245.11 25.4)
+		)
+		(stroke
+			(width 0)
+			(type default)
+		)
+	)
+	(wire
+		(pts
 			(xy 102.87 165.1) (xy 110.49 165.1)
 		)
@@
 	(symbol
 		(lib_id "power:GND")
+		(at 245.11 31.75 0)
+		(unit 1)
+		(body_style 1)
+		(exclude_from_sim no)
+		(in_bom yes)
+		(on_board yes)
+		(in_pos_files yes)
+		(dnp no)
+		(fields_autoplaced yes)
+		(property "Reference" "#PWR07"
+			(at 245.11 38.1 0)
+			(hide yes)
+			(show_name no)
+			(do_not_autoplace no)
+			(effects
+				(font
+					(size 1.27 1.27)
+				)
+			)
+		)
+		(property "Value" "GND"
+			(at 245.11 36.83 0)
+			(show_name no)
+			(do_not_autoplace no)
+			(effects
+				(font
+					(size 1.27 1.27)
+				)
+			)
+		)
+		(property "Footprint" ""
+			(at 245.11 31.75 0)
+			(hide yes)
+			(show_name no)
+			(do_not_autoplace no)
+			(effects
+				(font
+					(size 1.27 1.27)
+				)
+			)
+		)
+		(property "Datasheet" ""
+			(at 245.11 31.75 0)
+			(hide yes)
+			(show_name no)
+			(do_not_autoplace no)
+			(effects
+				(font
+					(size 1.27 1.27)
+				)
+			)
+		)
+		(property "Description" "Power symbol creates a global label with name \"GND\" , ground"
+			(at 245.11 31.75 0)
+			(hide yes)
+			(show_name no)
+			(do_not_autoplace no)
+			(effects
+				(font
+					(size 1.27 1.27)
+				)
+			)
+		)
+		(pin "1"
+		)
+		(instances
+			(project "T41_2_lpf"
+				(path "/5fc700c6-272f-41b7-8650-23a96fb06ce8"
+					(reference "#PWR07")
+					(unit 1)
+				)
+			)
+		)
+	)
+	(symbol
+		(lib_id "power:GND")
 		(at 143.51 36.83 0)
 		(unit 1)
@@
 					(unit 1)
 				)
+			)
+		)
+	)
+	(symbol
+		(lib_id "Device:R_Small_US")
+		(at 245.11 27.94 180)
+		(unit 1)
+		(body_style 1)
+		(exclude_from_sim no)
+		(in_bom yes)
+		(on_board yes)
+		(in_pos_files yes)
+		(dnp no)
+		(property "Reference" "R7"
+			(at 241.554 26.924 0)
+			(show_name no)
+			(do_not_autoplace no)
+			(effects
+				(font
+					(size 1.27 1.27)
+				)
+			)
+		)
+		(property "Value" "100k"
+			(at 241.3 29.718 0)
+			(show_name no)
+			(do_not_autoplace no)
+			(effects
+				(font
+					(size 1.27 1.27)
+				)
+			)
+		)
+		(property "Footprint" "Resistor_SMD:R_1206_3216Metric"
+			(at 245.11 27.94 0)
+			(hide yes)
+			(show_name no)
+			(do_not_autoplace no)
+			(effects
+				(font
+					(size 1.27 1.27)
+				)
+			)
+		)
+		(property "Datasheet" ""
+			(at 245.11 27.94 0)
+			(hide yes)
+			(show_name no)
+			(do_not_autoplace no)
+			(effects
+				(font
+					(size 1.27 1.27)
+				)
+			)
+		)
+		(property "Description" "Resistor, small US symbol"
+			(at 245.11 27.94 0)
+			(hide yes)
+			(show_name no)
+			(do_not_autoplace no)
+			(effects
+				(font
+					(size 1.27 1.27)
+				)
+			)
+		)
+		(pin "2"
+		)
+		(pin "1"
+		)
+		(instances
+			(project "T41_2_lpf"
+				(path "/5fc700c6-272f-41b7-8650-23a96fb06ce8"
+					(reference "R7")
+					(unit 1)
+				)
