File: T41_2_lpf.kicad_sch (KiCad schematic)
At the start: 37 parts, among them J1 5-1814832-1, J2 5-1814832-1, J3 5-1814832-1, J4 Conn_02x08_Odd_Even, J5 Conn_02x05_Odd_Even, J6 B2B-XH-A_LF__SN_, Q6 Q_NMOS_GSD, U12 4002, U13 TCA9534

Commit message: Added bypass capacitor to TXRX.  Did not uprev.
Parts:
- added C70: 0.01uF, Capacitor_SMD:C_1206_3216Metric, symbol Device:C_Small
Connections:
- net GND: now also C70.2
- net TXRX: now also C70.1
Changed lines of the file:
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@@
 	)
 	(junction
+		(at 41.275 153.67)
+		(diameter 0)
+		(color 0 0 0 0)
+	)
+	(junction
 		(at 232.41 52.07)
 		(diameter 0)
@@
 	(wire
 		(pts
-			(xy 39.37 153.67) (xy 53.34 153.67)
+			(xy 39.37 153.67) (xy 41.275 153.67)
 		)
 		(stroke
@@
 	(wire
 		(pts
+			(xy 41.275 156.21) (xy 41.275 153.67)
+		)
+		(stroke
+			(width 0)
+			(type default)
+		)
+	)
+	(wire
+		(pts
 			(xy 207.01 60.96) (xy 212.09 60.96)
 		)
@@
 	(wire
 		(pts
+			(xy 41.275 153.67) (xy 53.34 153.67)
+		)
+		(stroke
+			(width 0)
+			(type default)
+		)
+	)
+	(wire
+		(pts
 			(xy 53.34 156.21) (xy 53.34 158.75)
 		)
@@
 	(wire
 		(pts
+			(xy 41.275 161.29) (xy 41.275 162.56)
+		)
+		(stroke
+			(width 0)
+			(type default)
+		)
+	)
+	(wire
+		(pts
 			(xy 73.66 127) (xy 80.01 127)
 		)
@@
 	)
 	(symbol
+		(lib_id "Device:C_Small")
+		(at 41.275 158.75 0)
+		(unit 1)
+		(body_style 1)
+		(exclude_from_sim no)
+		(in_bom yes)
+		(on_board yes)
+		(in_pos_files yes)
+		(dnp no)
+		(fields_autoplaced yes)
+		(property "Reference" "C70"
+			(at 44.45 157.4862 0)
+			(show_name no)
+			(do_not_autoplace no)
+			(effects
+				(font
+					(size 1.27 1.27)
+				)
+				(justify left)
+			)
+		)
+		(property "Value" "0.01uF"
+			(at 44.45 160.0262 0)
+			(show_name no)
+			(do_not_autoplace no)
+			(effects
+				(font
+					(size 1.27 1.27)
+				)
+				(justify left)
+			)
+		)
+		(property "Footprint" "Capacitor_SMD:C_1206_3216Metric"
+			(at 41.275 158.75 0)
+			(hide yes)
+			(show_name no)
+			(do_not_autoplace no)
+			(effects
+				(font
+					(size 1.27 1.27)
+				)
+			)
+		)
+		(property "Datasheet" ""
+			(at 41.275 158.75 0)
+			(hide yes)
+			(show_name no)
+			(do_not_autoplace no)
+			(effects
+				(font
+					(size 1.27 1.27)
+				)
+			)
+		)
+		(property "Description" "Unpolarized capacitor, small symbol"
+			(at 41.275 158.75 0)
+			(hide yes)
+			(show_name no)
+			(do_not_autoplace no)
+			(effects
+				(font
+					(size 1.27 1.27)
+				)
+			)
+		)
+		(pin "2"
+		)
+		(pin "1"
+		)
+		(instances
+			(project "T41_2_lpf"
+				(path "/5fc700c6-272f-41b7-8650-23a96fb06ce8"
+					(reference "C70")
+					(unit 1)
+				)
+			)
+		)
+	)
+	(symbol
 		(lib_id "Device:L")
 		(at 97.79 52.07 0)
@@
 					(unit 1)
 				)
+			)
+		)
+	)
+	(symbol
+		(lib_id "power:GND")
+		(at 41.275 162.56 0)
+		(unit 1)
+		(body_style 1)
+		(exclude_from_sim no)
+		(in_bom yes)
+		(on_board yes)
+		(in_pos_files yes)
+		(dnp no)
+		(property "Reference" "#PWR050"
+			(at 41.275 168.91 0)
+			(hide yes)
+			(show_name no)
+			(do_not_autoplace no)
+			(effects
+				(font
+					(size 1.27 1.27)
+				)
+			)
+		)
+		(property "Value" "GND"
+			(at 45.085 163.83 0)
+			(show_name no)
+			(do_not_autoplace no)
+			(effects
+				(font
+					(size 1.27 1.27)
+				)
+			)
+		)
+		(property "Footprint" ""
+			(at 41.275 162.56 0)
+			(hide yes)
+			(show_name no)
+			(do_not_autoplace no)
+			(effects
+				(font
+					(size 1.27 1.27)
+				)
+			)
+		)
+		(property "Datasheet" ""
+			(at 41.275 162.56 0)
+			(hide yes)
+			(show_name no)
+			(do_not_autoplace no)
+			(effects
+				(font
+					(size 1.27 1.27)
+				)
+			)
+		)
+		(property "Description" "Power symbol creates a global label with name \"GND\" , ground"
+			(at 41.275 162.56 0)
+			(hide yes)
+			(show_name no)
+			(do_not_autoplace no)
+			(effects
+				(font
+					(size 1.27 1.27)
+				)
+			)
+		)
+		(pin "1"
+		)
+		(instances
+			(project "T41_2_lpf"
+				(path "/5fc700c6-272f-41b7-8650-23a96fb06ce8"
+					(reference "#PWR050")
+					(unit 1)
+				)
